File: pcb/steel-toe.kicad_pcb (KiCad board)
At the start: 2 copper layers, 133.7 x 81.8 mm, 33 parts, among them J0 AudioJack4dpb, SW1 SW_Push, SW10 SW_Push, SW11 SW_Push, SW12 SW_Push, SW13 SW_Push, SW14 SW_Push, SW15 SW_Push, SW16 SW_Push, SW17 SW_Push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

Commit message: Use reversible pro-micro footprint and other BoardSource components (#1)
* updated pcb to how I wanted it and made readme not shit

* forgot to save

* git ignore
Parts:
- SW18, SW21: footprint footprints:reset-switch-angled-4pin -> bs_lib:smd_rst_sw
- U1: footprint footprints:pro-micro -> bs_lib:ProMicro_facedown_new_dual
- turned U1 to -90 degrees
Routing:
- net K10: track 50.5 -> 32.9 mm
- net K11: track 144.7 -> 127.3 mm, vias 1 -> 2
- net K12: track 116.9 -> 101.5 mm, vias 1 -> 2
- net K15: track 51.2 -> 35.9 mm, vias 1 -> 2
- net K13: track 91.9 -> 78.8 mm, vias 1 -> 2
- net K9: track 79.4 -> 66.9 mm, vias 2 -> 3
- net K14: track 70.9 -> 59.2 mm, vias 1 -> 2
- net K16: track 74.5 -> 63.6 mm, vias 1 -> 2
- net VCC: track 32.5 -> 43.1 mm, vias 0 -> 1
- net K4: track 16.7 -> 25.8 mm
- net K17: track 65.3 -> 58.1 mm
- net SERIAL: track 35.5 -> 40.6 mm
- net K3: track 36.2 -> 39.9 mm
- net K2: track 57.0 -> 59.9 mm
- net K8: track 61.7 -> 64.4 mm
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Other:
- board text added: "Install Pro-Micro Face Down Jump bottom side jumpers"
