File: pcb/steel-toe.kicad_sch (KiCad schematic)
At the start: 25 parts, among them J0 AudioJack4dpb, SW1 SW_Push, SW10 SW_Push, SW11 SW_Push, SW12 SW_Push, SW13 SW_Push, SW14 SW_Push, SW15 SW_Push, SW16 SW_Push, SW17 SW_Push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

Commit message: Use reversible pro-micro footprint and other BoardSource components (#1)
* updated pcb to how I wanted it and made readme not shit

* forgot to save

* git ignore
Parts:
- SW18, SW21: footprint footprints:reset-switch-angled-4pin -> bs_lib:smd_rst_sw
- U1: footprint footprints:pro-micro -> bs_lib:ProMicro_facedown_new_dual
